File: hw/esp32c3_cc1101_dongle.kicad_pcb (KiCad board)
At the start: 2 copper layers, 60 x 24 mm, 7 parts

Commit message: Update carrier PCB to v1.2: trimmed USB edge, antenna keepout, logo
- Trim board outline flush to the ESP32 module's edge so its onboard
  USB-C connector overhangs the carrier board, matching the new case
  design; port-adjacent mounting holes relocated and verified clear of
  copper.
- Replace the 4 uniform mounting holes with 6 in three roles (far,
  middle, near-USB) matching the reworked case standoffs, each checked
  against real routed trace/pad positions rather than eyeballed.
- Add a full ground-plane keepout under the ESP32 module's antenna,
  sized to its own footprint so the pour stays naturally continuous at
  the board edges (no bridge vias needed).
- Fix silkscreen: swap the pin-1 square marker from 5V to GND, tidy
  GPIO/power label placement and edge clearance, add a "BB" logo.
- Export the two custom footprints (ESP32 socket, CC1101 header) to a
  real Custom_Library.pretty + fp-lib-table so KiCad can resolve them
  instead of only the board's embedded copies.
- Bump silkscreen version label to v1.2.

Verified throughout with kicad-cli: 0 DRC errors, ground continuity
confirmed via the DRC unconnected-items check after the keepout change.

Co-Authored-By: Claude Sonnet 5 <noreply@anthropic.com>
Parts:
- removed the ? at (52.5, 58.5)
- removed the ? at (52.5, 41.5)
- added ?: , MountingHole:MountingHole_2.5mm, F.Cu at (57.5, 46.0)
- added ?: , MountingHole:MountingHole_2.5mm, F.Cu at (57.5, 54.0)
- added ?: , MountingHole:MountingHole_2.5mm, F.Cu at (81.0, 42.5)
- added ?: , MountingHole:MountingHole_2.5mm, F.Cu at (81.0, 59.2)
- added ?: LOGO, LOGO, B.Cu at (105.2, 50.1)
Other:
- board size 60 x 24 mm -> 56.2 x 24 mm
- board text added: "github.com/bradrblack/rf-ceiling-fan-remote v1.2"
- board text removed: "github.com/bradrblack/rf-ceiling-fan-remote v1.1"
